Commit message: Refactor environment hooks and update world definitions for nova_gazebo

File: src/nova_description/urdf/Nova2.urdf.xacro (robot description, xacro)
@@ -3,7 +3,7 @@
   <xacro:arg name="name" default="nova2_robot"/>
   <xacro:arg name="use_ros2_control" default="true"/>
-  <ros>
-    <namespace>${robot_name}</namespace>
-  </ros>
+  <!-- <ros>
+    <namespace>${name}</namespace>
+  </ros> -->
   <xacro:include filename="$(find nova_description)/urdf/nova2.gazebo" />
   <!-- ===== World / dummy / base ===== -->

File: src/nova_gazebo/worlds/my_world.sdf.xacro (robot description, xacro)
@@ -10,4 +10,8 @@
   <xacro:property name="platform_base_height" value="0.35"/>
   <xacro:property name="initial_x" value="0.15"/>
+  <xacro:property name="initial_y_cube0" value="1.8"/>
+  <xacro:property name="initial_y_cube1" value="1.6"/>
+  <xacro:property name="initial_y_cube2" value="1.4"/>
+  <xacro:property name="initial_y_cube3" value="1.2"/>
   <!-- Reusable macro to include a model with pose -->
 <xacro:macro name="spawn_model" params="name uri x y z roll pitch yaw static:=true">
@@ -67,5 +71,5 @@
         name="container_l"
         uri="${container_l_uri}"
-        x="${initial_x}" y="0" z="${0.11+platform_base_height}"
+        x="${initial_x}" y="${initial_y_cube0}" z="${0.11+platform_base_height}"
         roll="0" pitch="0" yaw="0"
         static="false"/>
@@ -73,5 +77,5 @@
         name="container_m"
         uri="${container_m_uri}"
-        x="${initial_x}" y="0" z="${0.12+platform_base_height}"
+        x="${initial_x}" y="${initial_y_cube0}" z="${0.12+platform_base_height}"
         roll="0" pitch="0" yaw="0"
         static="false"/>
@@ -79,5 +83,5 @@
         name="object"
         uri="${object_uri}"
-        x="${initial_x}" y="0" z="${0.13+platform_base_height}"
+        x="${initial_x}" y="${initial_y_cube0}" z="${0.13+platform_base_height}"
         roll="0" pitch="0" yaw="0"
         static="false"/>
@@ -107,7 +111,25 @@
         static="true"/>
     <xacro:spawn_model
-        name="sliding_cube"
+        name="sliding_cube0"
         uri="${sliding_cube_uri}"
-        x="${initial_x}" y="0" z="${0.1+platform_base_height}"
+        x="${initial_x}" y="${initial_y_cube0}" z="${0.1+platform_base_height}"
+        roll="0" pitch="0" yaw="0"
+        static="false"/>
+    <xacro:spawn_model
+        name="sliding_cube1"
+        uri="${sliding_cube_uri}"
+        x="${initial_x}" y="${initial_y_cube1}" z="${0.1+platform_base_height}"
+        roll="0" pitch="0" yaw="0"
+        static="false"/>
+    <xacro:spawn_model
+        name="sliding_cube2"
+        uri="${sliding_cube_uri}"
+        x="${initial_x}" y="${initial_y_cube2}" z="${0.1+platform_base_height}"
+        roll="0" pitch="0" yaw="0"
+        static="false"/>
+    <xacro:spawn_model
+        name="sliding_cube3"
+        uri="${sliding_cube_uri}"
+        x="${initial_x}" y="${initial_y_cube3}" z="${0.1+platform_base_height}"
         roll="0" pitch="0" yaw="0"
         static="false"/>

Commit message: fix one namespace robot controller

File: src/nova_description/urdf/Nova2.urdf.xacro (robot description, xacro)
@@ -3,8 +3,5 @@
   <xacro:arg name="name" default="nova2_robot"/>
   <xacro:arg name="use_ros2_control" default="true"/>
-  <!-- <ros>
-    <namespace>${name}</namespace>
-  </ros> -->
-  <xacro:include filename="$(find nova_description)/urdf/nova2.gazebo" />
+  <xacro:include filename="$(find nova_description)/urdf/nova2.gazebo.xacro" />
   <!-- ===== World / dummy / base ===== -->
   <link name="dummy_link"/>
@@ -59,5 +56,5 @@
     <child  link="Link1"/>
     <axis xyz="0 0 -1"/>
-    <limit lower="-6.28" upper="6.28" effort="300" velocity="100"/>
+    <limit lower="-6.28" upper="6.28" effort="300" velocity="200"/>
   </joint>
   <link name="Link2">
@@ -83,5 +80,5 @@
     <child  link="Link2"/>
     <axis xyz="0 0 1"/>
-    <limit lower="-3.14" upper="3.14" effort="300" velocity="100"/>
+    <limit lower="-3.14" upper="3.14" effort="300" velocity="200"/>
   </joint>
   <link name="Link3">
@@ -107,5 +104,5 @@
     <child  link="Link3"/>
     <axis xyz="0 0 1"/>
-    <limit lower="-2.79" upper="2.79" effort="300" velocity="100"/>
+    <limit lower="-2.79" upper="2.79" effort="300" velocity="200"/>
   </joint>
   <link name="Link4">
@@ -131,5 +128,5 @@
     <child  link="Link4"/>
     <axis xyz="0 0 -1"/>
-    <limit lower="-6.28" upper="6.28" effort="300" velocity="100"/>
+    <limit lower="-6.28" upper="6.28" effort="300" velocity="200"/>
   </joint>
   <link name="Link5">
@@ -154,5 +151,5 @@
     <child  link="Link5"/>
     <axis xyz="0 0 -1"/>
-    <limit lower="-6.28" upper="6.28" effort="300" velocity="100"/>
+    <limit lower="-6.28" upper="6.28" effort="300" velocity="200"/>
   </joint>
   <link name="Link6">
@@ -177,13 +174,13 @@
     <child  link="Link6"/>
     <axis xyz="0 0 1"/>
-    <limit lower="-6.28" upper="6.28" effort="300" velocity="100"/>
+    <limit lower="-6.28" upper="6.28" effort="300" velocity="200"/>
   </joint>
   <!-- ===== Gazebo per-link visual materials (Gazebo Classic 可见；RViz不受影响) ===== -->
-  <gazebo reference="base_link"><gravity>false</gravity><selfCollide>true</selfCollide><material></material></gazebo>
-  <gazebo reference="Link1"><gravity>false</gravity><selfCollide>true</selfCollide><material></material></gazebo>
-  <gazebo reference="Link2"><gravity>false</gravity><selfCollide>true</selfCollide><material></material></gazebo>
-  <gazebo reference="Link3"><gravity>false</gravity><selfCollide>true</selfCollide><material></material></gazebo>
-  <gazebo reference="Link4"><gravity>false</gravity><selfCollide>true</selfCollide><material></material></gazebo>
-  <gazebo reference="Link5"><gravity>false</gravity><selfCollide>true</selfCollide><material></material></gazebo>
-  <gazebo reference="Link6"><gravity>false</gravity><selfCollide>true</selfCollide><material></material></gazebo>
+  <gazebo reference="base_link"><gravity>true</gravity><selfCollide>true</selfCollide><material></material></gazebo>
+  <gazebo reference="Link1"><gravity>true</gravity><selfCollide>true</selfCollide><material></material></gazebo>
+  <gazebo reference="Link2"><gravity>true</gravity><selfCollide>true</selfCollide><material></material></gazebo>
+  <gazebo reference="Link3"><gravity>true</gravity><selfCollide>true</selfCollide><material></material></gazebo>
+  <gazebo reference="Link4"><gravity>true</gravity><selfCollide>true</selfCollide><material></material></gazebo>
+  <gazebo reference="Link5"><gravity>true</gravity><selfCollide>true</selfCollide><material></material></gazebo>
+  <gazebo reference="Link6"><gravity>true</gravity><selfCollide>true</selfCollide><material></material></gazebo>
 </robot>

Commit message: Update robot controller configurations and launch files for nova2 robots

File: src/nova_description/urdf/Nova2.urdf.xacro (robot description, xacro)
@@ -3,5 +3,6 @@
   <xacro:arg name="name" default="nova2_robot"/>
   <xacro:arg name="use_ros2_control" default="true"/>
-  <xacro:include filename="$(find nova_description)/urdf/nova2.gazebo.xacro" />
+  <xacro:arg name="ns"   default="nova2_robot0"/>
+  <xacro:arg name="use_ros2_control" default="true"/>
   <!-- ===== World / dummy / base ===== -->
   <link name="dummy_link"/>
@@ -184,3 +185,73 @@
   <gazebo reference="Link5"><gravity>true</gravity><selfCollide>true</selfCollide><material></material></gazebo>
   <gazebo reference="Link6"><gravity>true</gravity><selfCollide>true</selfCollide><material></material></gazebo>
+    <!-- ros_control plugin -->
+    <gazebo>
+      <plugin
+        filename="gz_ros2_control-system"
+        name="gz_ros2_control::GazeboSimROS2ControlPlugin">
+        <!-- your controllers YAML -->
+        <parameters>$(find nova_description)/config/nova2_controllers.yaml</parameters>
+        <!-- this is where the namespace is used -->
+        <ros>
+          <namespace>$(arg ns)</namespace>
+          <!-- <remapping>/tf:=/${ns}/tf</remapping>  optional -->
+        </ros>
+      </plugin>
+    </gazebo>
+    <!-- joint_state_publisher from Gazebo (optional but handy) -->
+    <gazebo>
+      <plugin
+        filename="gz-sim-joint-state-publisher-system"
+        name="gz::sim::systems::JointStatePublisher">
+        <topic>joint_states</topic>
+        <joint_name>joint1</joint_name>
+        <joint_name>joint2</joint_name>
+        <joint_name>joint3</joint_name>
+        <joint_name>joint4</joint_name>
+        <joint_name>joint5</joint_name>
+        <joint_name>joint6</joint_name>
+      </plugin>
+    </gazebo>
+    <!-- ros2_control hardware description -->
+    <ros2_control name="GazeboSimSystem" type="system">
+      <hardware>
+        <plugin>gz_ros2_control/GazeboSimSystem</plugin>
+      </hardware>
+      <joint name="joint1">
+        <command_interface name="position"/>
+        <state_interface name="position">
+          <param name="initial_value">0.0</param>
+        </state_interface>
+      </joint>
+      <joint name="joint2">
+        <command_interface name="position"/>
+        <state_interface name="position">
+          <param name="initial_value">0.0</param>
+        </state_interface>
+      </joint>
+      <joint name="joint3">
+        <command_interface name="position"/>
+        <state_interface name="position">
+          <param name="initial_value">0.0</param>
+        </state_interface>
+      </joint>
+      <joint name="joint4">
+        <command_interface name="position"/>
+        <state_interface name="position">
+          <param name="initial_value">0.0</param>
+        </state_interface>
+      </joint>
+      <joint name="joint5">
+        <command_interface name="position"/>
+        <state_interface name="position">
+          <param name="initial_value">0.0</param>
+        </state_interface>
+      </joint>
+      <joint name="joint6">
+        <command_interface name="position"/>
+        <state_interface name="position">
+          <param name="initial_value">0.0</param>
+        </state_interface>
+      </joint>
+    </ros2_control>
 </robot>

File: src/nova_description/urdf/nova2.gazebo.xacro (robot description, xacro)
@@ -1,73 +1,77 @@
 <?xml version="1.0"?>
-<!--
-Copied and modified from ROS1 example -
-https://github.com/ros-simulation/gazebo_ros_demos/blob/kinetic-devel/nova2_robot0_description/urdf/nova2_robot0.gazebo
--->
-<robot xmlns:xacro="http://ros.org/wiki/xacro">
-  <!-- <xacro:macro name="nova2_gazebo"> -->
+<robot xmlns:xacro="http://www.ros.org/wiki/xacro">
+  <!-- Macro that injects Gazebo + ros2_control for this arm.
+       Parameter "ns" is the ROS namespace for this robot. -->
+  <xacro:macro name="nova2_gazebo" params="ns">
     <!-- ros_control plugin -->
     <gazebo>
-      <plugin filename="gz_ros2_control-system" name="gz_ros2_control::GazeboSimROS2ControlPlugin">
+      <plugin
+        filename="gz_ros2_control-system"
+        name="gz_ros2_control::GazeboSimROS2ControlPlugin">
+        <!-- your controllers YAML -->
         <parameters>$(find nova_description)/config/nova2_controllers.yaml</parameters>
+        <!-- this is where the namespace is used -->
         <ros>
-             <namespace>nova2_robot0</namespace>
-        <!-- <remapping>/tf:=/$(arg namespace)/tf</remapping> -->
-         </ros>
+          <namespace>${arg ns}</namespace>
+          <!-- <remapping>/tf:=/${ns}/tf</remapping>  optional -->
+        </ros>
       </plugin>
     </gazebo>
+    <!-- joint_state_publisher from Gazebo (optional but handy) -->
     <gazebo>
-        <plugin
-            filename="gz-sim-joint-state-publisher-system"
-            name="gz::sim::systems::JointStatePublisher">
-            <topic>joint_states</topic>
-            <joint_name>joint1</joint_name>
-            <joint_name>joint2</joint_name>
-            <joint_name>joint3</joint_name>
-            <joint_name>joint4</joint_name>
-            <joint_name>joint5</joint_name>
-            <joint_name>joint6</joint_name>
-        </plugin>
+      <plugin
+        filename="gz-sim-joint-state-publisher-system"
+        name="gz::sim::systems::JointStatePublisher">
+        <topic>joint_states</topic>
+        <joint_name>joint1</joint_name>
+        <joint_name>joint2</joint_name>
+        <joint_name>joint3</joint_name>
+        <joint_name>joint4</joint_name>
+        <joint_name>joint5</joint_name>
+        <joint_name>joint6</joint_name>
+      </plugin>
     </gazebo>
-   <ros2_control name="GazeboSimSystem" type="system">
-        <hardware>
-          <plugin>gz_ros2_control/GazeboSimSystem</plugin>
-        </hardware>
-        <joint name="joint1">
-            <command_interface name="position"/>
-            <state_interface name="position">
-                <param name="initial_value">0.0</param>
-            </state_interface>
-        </joint>
-        <joint name="joint2">
-            <command_interface name="position"/>
-            <state_interface name="position">
-                <param name="initial_value">0.0</param>
-            </state_interface>
-        </joint>
-        <joint name="joint3">
-            <command_interface name="position"/>
-            <state_interface name="position">
-                <param name="initial_value">0.0</param>
-            </state_interface>
-        </joint>
-        <joint name="joint4">
-            <command_interface name="position"/>
-            <state_interface name="position">
-                <param name="initial_value">0.0</param>
-            </state_interface>
-        </joint>
-        <joint name="joint5">
-            <command_interface name="position"/>
-            <state_interface name="position">
-                <param name="initial_value">0.0</param>
-            </state_interface>
-        </joint>
-        <joint name="joint6">
-            <command_interface name="position"/>
-            <state_interface name="position">
-                <param name="initial_value">0.0</param>
-            </state_interface>
-        </joint>
+    <!-- ros2_control hardware description -->
+    <ros2_control name="GazeboSimSystem" type="system">
+      <hardware>
+        <plugin>gz_ros2_control/GazeboSimSystem</plugin>
+      </hardware>
+      <joint name="joint1">
+        <command_interface name="position"/>
+        <state_interface name="position">
+          <param name="initial_value">0.0</param>
+        </state_interface>
+      </joint>
+      <joint name="joint2">
+        <command_interface name="position"/>
+        <state_interface name="position">
+          <param name="initial_value">0.0</param>
+        </state_interface>
+      </joint>
+      <joint name="joint3">
+        <command_interface name="position"/>
+        <state_interface name="position">
+          <param name="initial_value">0.0</param>
+        </state_interface>
+      </joint>
+      <joint name="joint4">
+        <command_interface name="position"/>
+        <state_interface name="position">
+          <param name="initial_value">0.0</param>
+        </state_interface>
+      </joint>
+      <joint name="joint5">
+        <command_interface name="position"/>
+        <state_interface name="position">
+          <param name="initial_value">0.0</param>
+        </state_interface>
+      </joint>
+      <joint name="joint6">
+        <command_interface name="position"/>
+        <state_interface name="position">
+          <param name="initial_value">0.0</param>
+        </state_interface>
+      </joint>
     </ros2_control>
-  <!-- </xacro:macro> -->
+  </xacro:macro>
 </robot>
